File: Kicad/1015-InpBrdG2/1015.sch (KiCad schematic (older format))
At the start: 10 parts, among them P1 TST, P2 CONN_4, P3 CONN_4, P4 CONN_6, P5 CONN_8, P6 CONN_4

Commit message: Updates to silkscreen and created mashup.  These Gerbers sent to PCB house.
Parts:
- R1: value 100K -> 0
Changed lines of the file:
@@
 LIBS:contrib
 LIBS:valves
+LIBS:1015-cache
 EELAYER 27 0
 EELAYER END
@@
 Sheet 1 1
 Title "Input Board (Gen 2)"
-Date "26 jul 2015"
+Date "28 jul 2015"
 Rev "-"
 Comp "Open Pinball Project"
@@
 P 3350 5600
 F 0 "R1" V 3430 5600 40  0000 C CNN
-F 1 "100K" V 3357 5601 40  0000 C CNN
+F 1 "0" V 3357 5601 40  0000 C CNN
 F 2 "~" V 3280 5600 30  0000 C CNN
 F 3 "~" H 3350 5600 30  0000 C CNN
