File: Kicad/1013-SolDrvG2/1013.sch (KiCad schematic (older format))
At the start: 16 parts, among them P1 TST, P10 SPADE_187, P2 CONN_4, P3 CONN_4, P4 CONN2X3MOLEX, P5 CONN_4, P6 CONN_8, Q1 MOSFET_N, Q2 MOSFET_N, Q3 MOSFET_N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

Commit message: Updates to silkscreen and created mashup.  These Gerbers sent to PCB house.
Parts:
- R1: value 100K -> 0
Changed lines of the file:
@@
 Sheet 1 1
 Title "Solenoid Driver (Gen 2)"
-Date "24 jul 2015"
+Date "28 jul 2015"
 Rev "-"
 Comp "Open Pinball Project"
@@
 P 3150 3900
 F 0 "R1" V 3230 3900 40  0000 C CNN
-F 1 "100K" V 3157 3901 40  0000 C CNN
+F 1 "0" V 3157 3901 40  0000 C CNN
 F 2 "~" V 3080 3900 30  0000 C CNN
 F 3 "~" H 3150 3900 30  0000 C CNN

Commit message: Rename 1012-InpSolGen2 to 1012-STM32F0InpSol to indicate it is for the STM32F0 Discovery board.  1012 is an untested and orphaned set of boards.  Rename 1015-InpBrdG2 to 1015-SpiNeoPxl.  1015 basically has a single pin used for connecting to Neopixels using the SPI bus.  Newer version uses the internal FPGA of the PSOC 4200 and uses a different output pin.  1015 is tested, but mostly orphaned since the FPGA version uses less memory and processing.
Update 1013-SolDrvG2, 1014-IncandBrdG2, and 1016-IntfBrdG2 to version 4.0.7 of KiCad.  Required updating the gnd and resistor symbols to match the new standard libraries.
Parts:
- P10: symbol SPADE_187 -> spade_187
- P4: symbol CONN2X3MOLEX -> CONN2x3Molex
- R1, R2, R3, R4, R5: footprint ~ -> (none)
