File: Kicad/1014-IncandBrdG2/1014.sch (KiCad schematic (older format))
At the start: 24 parts, among them P1 TST, P2 CONN_4, P3 CONN_4, P4 SPADE_187, P5 CONN_8, P6 CONN_2, P7 CONN_8, Q1 MOSFET_N, Q2 MOSFET_N, Q3 MOSFET_N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

Commit message: Updates to silkscreen and created mashup.  These Gerbers sent to PCB house.
Parts:
- R1: value 100K -> 0
Changed lines of the file:
@@
 Sheet 1 1
 Title "Incandescent Driver (Gen 2)"
-Date "26 jul 2015"
+Date "28 jul 2015"
 Rev "-"
 Comp "Open Pinball Project"
@@
 P 2050 3000
 F 0 "R1" V 2130 3000 40  0000 C CNN
-F 1 "100K" V 2057 3001 40  0000 C CNN
+F 1 "0" V 2057 3001 40  0000 C CNN
 F 2 "~" V 1980 3000 30  0000 C CNN
 F 3 "~" H 2050 3000 30  0000 C CNN

Commit message: Fix labeling issue on the incandescent board.
Parts:
- removed R1: 0, ~, symbol R
Connections:
- net labels added: +VLED
- net labels removed: GNDPWR
- wire segments 123 -> 108
Other:
- moved on the sheet: P6, P7, Q1, Q2, Q3, Q4, Q5, Q6, Q7, Q8

Commit message: Rename 1012-InpSolGen2 to 1012-STM32F0InpSol to indicate it is for the STM32F0 Discovery board.  1012 is an untested and orphaned set of boards.  Rename 1015-InpBrdG2 to 1015-SpiNeoPxl.  1015 basically has a single pin used for connecting to Neopixels using the SPI bus.  Newer version uses the internal FPGA of the PSOC 4200 and uses a different output pin.  1015 is tested, but mostly orphaned since the FPGA version uses less memory and processing.
Update 1013-SolDrvG2, 1014-IncandBrdG2, and 1016-IntfBrdG2 to version 4.0.7 of KiCad.  Required updating the gnd and resistor symbols to match the new standard libraries.
Parts:
- P4: symbol SPADE_187 -> spade_187
- R2, R3, R4, R5, R6, R7, R8, R9: footprint ~ -> (none)
Changed lines of the file:
@@
 EESchema Schematic File Version 2
+LIBS:1014-rescue
 LIBS:commonpart
 LIBS:power
@@
 LIBS:memory
 LIBS:xilinx
-LIBS:special
 LIBS:microcontrollers
 LIBS:dsp
@@
 LIBS:valves
 LIBS:1014-cache
-EELAYER 27 0
+EELAYER 25 0
 EELAYER END
 $Descr A 11000 8500
@@
 $EndComp
 $Comp
-L SPADE_187 P4
+L spade_187 P4
 U 1 1 4F789F3A
 P 3100 3300
@@
 $EndComp
 $Comp
-L GND #PWR03
-U 1 1 55B16408
-P 2500 3200
-F 0 "#PWR03" H 2500 3200 30  0001 C CNN
-F 1 "GND" H 2500 3130 30  0001 C CNN
-F 2 "" H 2500 3200 60  0001 C CNN
-F 3 "" H 2500 3200 60  0001 C CNN
-	1    2500 3200
-	1    0    0    -1
-$EndComp
-$Comp
 L +12V1 #PWR04
 U 1 1 55B165D8
@@
 Wire Wire Line
 	1900 2600 1600 2600
-$Comp
-L R R2
-U 1 1 55B1776F
-P 3700 3250
-F 0 "R2" V 3780 3250 40  0000 C CNN
-F 1 "10K" V 3707 3251 40  0000 C CNN
-F 2 "~" V 3630 3250 30  0000 C CNN
-F 3 "~" H 3700 3250 30  0000 C CNN
-	1    3700 3250
-	-1   0    0    1
-$EndComp
 Wire Wire Line
 	6200 2200 6000 2200
@@
 $EndComp
 $Comp
-L R R3
-U 1 1 55B4EEBA
-P 4400 3250
-F 0 "R3" V 4480 3250 40  0000 C CNN
-F 1 "10K" V 4407 3251 40  0000 C CNN
-F 2 "~" V 4330 3250 30  0000 C CNN
-F 3 "~" H 4400 3250 30  0000 C CNN
-	1    4400 3250
-	-1   0    0    1
-$EndComp
-$Comp
 L MOSFET_N Q3
 U 1 1 55B4EEC4
@@
 $EndComp
 $Comp
-L R R4
-U 1 1 55B4EECA
-P 5100 3250
-F 0 "R4" V 5180 3250 40  0000 C CNN
-F 1 "10K" V 5107 3251 40  0000 C CNN
-F 2 "~" V 5030 3250 30  0000 C CNN
-F 3 "~" H 5100 3250 30  0000 C CNN
-	1    5100 3250
-	-1   0    0    1
-$EndComp
-$Comp
 L MOSFET_N Q4
 U 1 1 55B4EED4
@@
 $EndComp
 $Comp
-L R R5
-U 1 1 55B4EEDA
-P 5800 3250
-F 0 "R5" V 5880 3250 40  0000 C CNN
-F 1 "10K" V 5807 3251 40  0000 C CNN
-F 2 "~" V 5730 3250 30  0000 C CNN
-F 3 "~" H 5800 3250 30  0000 C CNN
-	1    5800 3250
-	-1   0    0    1
-$EndComp
-$Comp
 L MOSFET_N Q5
 U 1 1 55B4EEE4
@@
 $EndComp
 $Comp
-L R R6
-U 1 1 55B4EEEA
-P 6500 3250
-F 0 "R6" V 6580 3250 40  0000 C CNN
-F 1 "10K" V 6507 3251 40  0000 C CNN
-F 2 "~" V 6430 3250 30  0000 C CNN
-F 3 "~" H 6500 3250 30  0000 C CNN
-	1    6500 3250
-	-1   0    0    1
-$EndComp
-$Comp
 L MOSFET_N Q6
 U 1 1 55B4EEF4
@@
 $EndComp
 $Comp
-L R R7
-U 1 1 55B4EEFA
-P 7200 3250
-F 0 "R7" V 7280 3250 40  0000 C CNN
-F 1 "10K" V 7207 3251 40  0000 C CNN
-F 2 "~" V 7130 3250 30  0000 C CNN
-F 3 "~" H 7200 3250 30  0000 C CNN
-	1    7200 3250
-	-1   0    0    1
-$EndComp
-$Comp
 L MOSFET_N Q7
 U 1 1 55B4EF04
@@
 $EndComp
 $Comp
-L R R8
-U 1 1 55B4EF0A
-P 7900 3250
-F 0 "R8" V 7980 3250 40  0000 C CNN
-F 1 "10K" V 7907 3251 40  0000 C CNN
-F 2 "~" V 7830 3250 30  0000 C CNN
-F 3 "~" H 7900 3250 30  0000 C CNN
-	1    7900 3250
-	-1   0    0    1
-$EndComp
-$Comp
 L MOSFET_N Q8
 U 1 1 55B4EF14
@@
 	1    0    0    -1
 $EndComp
-$Comp
-L R R9
-U 1 1 55B4EF1A
-P 8600 3250
-F 0 "R9" V 8680 3250 40  0000 C CNN
-F 1 "10K" V 8607 3251 40  0000 C CNN
-F 2 "~" V 8530 3250 30  0000 C CNN
-F 3 "~" H 8600 3250 30  0000 C CNN
-	1    8600 3250
-	-1   0    0    1
-$EndComp
 Wire Wire Line
 	3500 1500 3500 4000
@@
 	3500 4000 3800 4000
 Wire Wire Line
-	3700 3500 3700 4000
+	3700 3400 3700 4000
 Connection ~ 3700 4000
 Wire Wire Line
@@
 	4200 4000 4500 4000
 Wire Wire Line
-	4400 3500 4400 4000
+	4400 3400 4400 4000
 Connection ~ 4400 4000
 Wire Wire Line
@@
 	4900 4000 5200 4000
 Wire Wire Line
-	5100 3500 5100 4000
+	5100 3400 5100 4000
 Connection ~ 5100 4000
 Wire Wire Line
@@
 	5600 4000 5900 4000
 Wire Wire Line
-	5800 3500 5800 4000
+	5800 3400 5800 4000
 Connection ~ 5800 4000
 Wire Wire Line
@@
 	7000 4000 7300 4000
 Wire Wire Line
-	7200 3500 7200 4000
+	7200 3400 7200 4000
 Connection ~ 7200 4000
 Wire Wire Line
@@
 	7700 4000 8000 4000
 Wire Wire Line
-	7900 3500 7900 4000
+	7900 3400 7900 4000
 Connection ~ 7900 4000
 Wire Wire Line
@@
 	8400 4000 8700 4000
 Wire Wire Line
-	8600 3500 8600 4000
+	8600 3400 8600 4000
 Connection ~ 8600 4000
 $Comp
@@
 $EndComp
 Wire Wire Line
-	3700 2800 3700 3000
+	3700 2800 3700 3100
 Wire Wire Line
 	3700 2900 8600 2900
 Wire Wire Line
-	4400 2900 4400 3000
+	4400 2900 4400 3100
 Connection ~ 3700 2900
 Wire Wire Line
-	5100 2900 5100 3000
+	5100 2900 5100 3100
 Connection ~ 4400 2900
 Wire Wire Line
-	5800 2900 5800 3000
+	5800 2900 5800 3100
 Connection ~ 5100 2900
 Wire Wire Line
-	6500 2900 6500 3000
+	6500 2900 6500 3100
 Connection ~ 5800 2900
 Wire Wire Line
-	7200 2900 7200 3000
+	7200 2900 7200 3100
 Connection ~ 6500 2900
 Wire Wire Line
-	7900 2900 7900 3000
+	7900 2900 7900 3100
 Connection ~ 7200 2900
 Wire Wire Line
-	8600 2900 8600 3000
+	8600 2900 8600 3100
 Connection ~ 7900 2900
 Wire Wire Line
@@
 	8300 4200 8300 5200
 Wire Wire Line
-	6500 3500 6500 4000
+	6500 3400 6500 4000
 Connection ~ 6500 4000
 $Comp
@@
 	1    0    0    -1
 $EndComp
+$Comp
+L GND #PWR?
+U 1 1 5A54FFE4
+P 2500 3200
+F 0 "#PWR?" H 2500 2950 50  0001 C CNN
+F 1 "GND" H 2500 3050 50  0000 C CNN
+F 2 "" H 2500 3200 50  0001 C CNN
+F 3 "" H 2500 3200 50  0001 C CNN
+	1    2500 3200
+	1    0    0    -1
+$EndComp
+$Comp
+L R R2
+U 1 1 5A5505AC
+P 3700 3250
+F 0 "R2" V 3780 3250 50  0000 C CNN
+F 1 "10K" V 3700 3250 50  0000 C CNN
+F 2 "" V 3630 3250 50  0001 C CNN
+F 3 "" H 3700 3250 50  0001 C CNN
+	1    3700 3250
+	1    0    0    -1
+$EndComp
+$Comp
+L R R3
+U 1 1 5A5507CD
+P 4400 3250
+F 0 "R3" V 4480 3250 50  0000 C CNN
+F 1 "10K" V 4400 3250 50  0000 C CNN
+F 2 "" V 4330 3250 50  0001 C CNN
+F 3 "" H 4400 3250 50  0001 C CNN
+	1    4400 3250
+	1    0    0    -1
+$EndComp
+$Comp
+L R R4
+U 1 1 5A55087D
+P 5100 3250
+F 0 "R4" V 5180 3250 50  0000 C CNN
+F 1 "10K" V 5100 3250 50  0000 C CNN
+F 2 "" V 5030 3250 50  0001 C CNN
+F 3 "" H 5100 3250 50  0001 C CNN
+	1    5100 3250
+	1    0    0    -1
+$EndComp
+$Comp
+L R R5
+U 1 1 5A5508F5
+P 5800 3250
+F 0 "R5" V 5880 3250 50  0000 C CNN
+F 1 "10K" V 5800 3250 50  0000 C CNN
+F 2 "" V 5730 3250 50  0001 C CNN
+F 3 "" H 5800 3250 50  0001 C CNN
+	1    5800 3250
+	1    0    0    -1
+$EndComp
+$Comp
+L R R6
+U 1 1 5A55098D
+P 6500 3250
+F 0 "R6" V 6580 3250 50  0000 C CNN
+F 1 "10K" V 6500 3250 50  0000 C CNN
+F 2 "" V 6430 3250 50  0001 C CNN
+F 3 "" H 6500 3250 50  0001 C CNN
+	1    6500 3250
+	1    0    0    -1
+$EndComp
+$Comp
+L R R7
+U 1 1 5A550A11
+P 7200 3250
+F 0 "R7" V 7280 3250 50  0000 C CNN
+F 1 "10K" V 7200 3250 50  0000 C CNN
+F 2 "" V 7130 3250 50  0001 C CNN
+F 3 "" H 7200 3250 50  0001 C CNN
+	1    7200 3250
+	1    0    0    -1
+$EndComp
+$Comp
+L R R8
+U 1 1 5A550AAF
+P 7900 3250
+F 0 "R8" V 7980 3250 50  0000 C CNN
+F 1 "10K" V 7900 3250 50  0000 C CNN
+F 2 "" V 7830 3250 50  0001 C CNN
+F 3 "" H 7900 3250 50  0001 C CNN
+	1    7900 3250
+	1    0    0    -1
+$EndComp
+$Comp
+L R R9
+U 1 1 5A550C1F
+P 8600 3250
+F 0 "R9" V 8680 3250 50  0000 C CNN
+F 1 "10K" V 8600 3250 50  0000 C CNN
+F 2 "" V 8530 3250 50  0001 C CNN
+F 3 "" H 8600 3250 50  0001 C CNN
+	1    8600 3250
+	1    0    0    -1
+$EndComp
